File: payload1_board/ocp.kicad_sch (KiCad schematic)
At the start: 13 parts, among them Q1 DTC114E, Q2 SSM6K403TU_LF, Q3 DTC114E, U6 LTC4361HTS8-2-TRMPBF

Commit message: LAST UPDATE
Parts:
- removed R5, R8: 100, Resistor_SMD:R_0805_2012Metric, symbol Device:R
- added R9: 100, symbol Device:R
- renumbered C46 to C11, C47 to C12, C48 to C13, D2 to D4, R3 to R7, R4 to R8, U6 to U1
Connections:
- net GND: now also R9.2
- net STM32_TO_OCP: now reaches Q1.1 (B), Q3.1 (B), SB16.1 (A)
- net at D4.1: now also R9.1
- net VDD renamed +3.3V
Other:
- moved on the sheet: C11, C12, C13, D4, Q2, Q3, R7, R8, SB16, U1
