File: payload1_board/sensores.kicad_sch (KiCad schematic)
At the start: 0 parts

Commit message: a
Parts:
- added C38: 100nf, symbol Device:C
- added C39, C42: 10uf, symbol Device:C
- added C40: 10nf, symbol Device:C
- added C41: 470nf, symbol Device:C
- added C43: 1uf, symbol Device:C
- added R2: 10k, symbol Device:R
- added U3: AIS328DQTR, QFPN24_4X4X1P8_STM, symbol AS328DQTR:AIS328DQTR
- added U4: MMC5983MA, MMC5983MA_MEM, symbol MMC5983MA:MMC5983MA
- added U5: I3G4250DTR, LGA-16_4X4X1_STM, symbol I3G4250DTR:I3G4250DTR
Connections:
- new net: C40.1, C41.1, U5.14 (PLLFILT)
- new net: C40.2, C41.2, R2.1
- new net: C38.1, C39.1, U3.5 (VDD)
- new net: C43.2, U4.2 (VDD)
- new net: C42.2, U4.10 (CAP)
- new net GND: C38.2, C39.2, C42.1, C43.1, R2.2, U3.10 (GND), U3.25 (GND), U3.6 (GND), U3.8 (GND), U3.9 (GND), U4.11 (GND), U4.9 (GND), U5.10 (RES), U5.11 (RES), U5.12 (RES), U5.13 (GND), U5.9 (RES)
