File: payload1_board/gps.kicad_sch (KiCad schematic)
At the start: 0 parts

Commit message: LAST UPDATE
Parts:
- added AE1: Antenna, symbol Device:Antenna
- added BT1: COIN_Cell, symbol Device:Battery_Cell
- added C42: 47pF, symbol Device:C
- added C43: 1.0uF, symbol Device:C
- added CR3: SD1206S040S1R0, SD1206_AVX, symbol SCHOTTKY_DIODE_SD1206S040S1R0:SD1206S040S1R0
- added D4: RED, symbol Device:LED
- added D5: YELLOW, symbol Device:LED
- added FL1: B39162B4348P810, B39162B4348P810, symbol GPS_SAW_FILTER_B39162B4348P810:B39162B4348P810
- added JP2, JP3: PWR, symbol Jumper:SolderJumper_2_Bridged
- added R11, R12, R13, R6, R7, R8: 33, symbol Device:R
- added R16: 3.3k, symbol Device:R
- added R17, R18: 1k, symbol Device:R
- added U1: MAX-M10S-00B, symbol MAX-M10S-00B:MAX-M10S-00B
Connections:
- new net: D5.2 (A), R18.2
- new net: AE1.1 (A), C42.1
- new net: C42.2, FL1.1 (INPUT)
- new net: CR3.1, R16.1
- new net: JP2.1 (A), R17.1
- new net: D4.2 (A), R17.2
- new net: JP3.1 (A), R18.1
- new net +3V3: CR3.2, JP2.2 (B), U1.7 (V_IO), U1.8 (VCC)
- new net GND: BT1.2 (-), C43.2, D4.1 (K), D5.1 (K), FL1.2 (GND1), FL1.3 (GND2), FL1.5 (GND3), U1.1 (GND), U1.10 (GND), U1.12 (GND)
- new net MAX_BACKUP: BT1.1 (+), C43.1, R16.2, U1.6 (V_BCKP)
- new net MAX_INT: R11.1, U1.5 (EXTINT)
- new net MAX_INT_TO_STM32: R11.2
- new net MAX_PPS: R12.1, U1.4 (TIMEPULSE)
- new net MAX_PPS_TO_STM32: JP3.2 (B), R12.2
- new net MAX_RESET_N: R6.1, U1.9 (~{RESET})
- new net MAX_RESET_N_TO_STM32: R6.2
- new net MAX_RF_IN: FL1.4 (OUTPUT), U1.11 (RF_IN)
- new net MAX_RXI: R8.1, U1.3 (RXD)
- new net MAX_RXI_TO_STM32: R8.2
- new net MAX_SAFE_N: R13.1, U1.18 (~{SAFEBOOT})
- new net MAX_SAFE_N_TO_STM32: R13.2
- new net MAX_TXO: R7.1, U1.2 (TXD)
- new net MAX_TXO_TO_STM32: R7.2
- no-connect marks 0 -> 7
Other:
- note added: "LNA AND ANTENNA"
- note added: "RTC BACKUP"
- note added: "SAW para antena pasiva. Poner LNA? Usar antena activa?"
- note added: "STAT LEDS"
