File: payload1_board/mcu.kicad_sch (KiCad schematic)
At the start: 34 parts, among them U1 STM32WLE5CCU6, Y1 32.768KHz, Y2 32MHz

Commit message: LAST UPDATE
Parts:
- removed C11, C12, C16, C7: 100nF, symbol Device:C
- removed C14: 0.47uF, symbol Device:C
- removed C32, C33, C34: 33pF, symbol Device:C
- removed C37: 4.7uF, symbol Device:C
- removed C6: 4.7nF, symbol Device:C
- removed D1: ESD, symbol Diode:ESD5Zxx
- removed L1: 600R@100MHz, symbol Device:FerriteBead_Small
- removed L2: 15uH, symbol Device:L
- removed SB1, SB11, SB13, SB14, SB2, SB7: Close, symbol Jumper:SolderJumper_2_Bridged
- removed SB8: Open, symbol Jumper:SolderJumper_2_Open
- removed U1: STM32WLE5CCU6, UFQFPN48_STM, symbol STM32WLE5:STM32WLE5CCU6
- removed Y1: 32.768KHz, symbol Device:Crystal_GND24_Small
- added D1: BLUE, symbol Device:LED
- added D2: RED, symbol Device:LED
- added FB1: 1k 100Mhz, symbol Device:FerriteBead
- added IC1: STM32F411CEU7, QFN50P700X700X65-49N-D, symbol STM32F411CEU7:STM32F411CEU7
- added J1: Screw_Terminal_01x04, symbol Connector:Screw_Terminal_01x04
- added J3: Screw_Terminal_01x02, symbol Connector:Screw_Terminal_01x02
- added R2, R4: 10K, symbol Device:R
- added R3: 10k, symbol Device:R
- added R5: 1.5k, symbol Device:R
- added R6: 5.1k, symbol Device:R
- added SW1, SW2, SW3: SW_SPST, symbol Switch:SW_SPST
- C1: value 4.7uF -> 100uF
- C10: value 4.7uF -> 2.2uF
- C6: renamed from C26; value 6.8pF -> 10pF
- C7: renamed from C31; value 6.8pF -> 10pF
- C8, C9: value 6.8pF -> 100nF
- R1: value 10K -> 330R
- Y2: value 32MHz -> 16MHz
Connections:
- net VBAT is gone; now on net GND: C1.2, C2.2, C3.2, C4.2, C5.2
- net ACCEL_CS_TO_STM_NSS: now also IC1.14 (PA4)
- net ACCEL_INT1_TO_STM: now also IC1.10 (PA0)
- net ACCEL_INT2_TO_STM: now also IC1.11 (PA1)
- net GND: now also C8.2, D2.1 (K), IC1.23 (VSS_1), IC1.35 (VSS_2), IC1.47 (VSS_3), IC1.49 (EP), IC1.8 (VSSA/VREF-), J1.4 (Pin_4), J3.1 (Pin_1), R3.2, R4.2, SW1.2 (B), SW2.2 (B); no longer C1.1, C2.1, C3.1, C4.1, C5.1, C8.1, R1.2
- net GYRO_CS_TO_STM_NSS: now also IC1.19 (PB1)
- net GYRO_INT1_TO_STM: now also IC1.12 (PA2)
- net GYRO_INT2_TO_STM: now also IC1.13 (PA3)
- net IMU_SCL_TO_STM_SCK: now also IC1.15 (PA5)
- net IMU_SDI_TO_STM_MOSI: now also IC1.17 (PA7)
- net IMU_SDO_TO_STM_MISO: now also IC1.16 (PA6)
- net MAG_CS_TO_STM_NSS: now also IC1.25 (PB12)
- net MAG_INT_TO_STM: now also IC1.31 (PA10)
- net NRST: now also C8.1, IC1.7 (NRST), R2.1, SW2.1 (A)
- net OSC_IN: now also C6.2, Y2.1, IC1.5 (PH0-OSC_IN)
- net OSC_OUT: now also C7.2, Y2.3, IC1.6 (PH1-OSC_OUT)
- net PA13: now also IC1.34 (PA13), J1.2 (Pin_2)
- net PC13: now also D1.1 (K), IC1.2 (PC13)
- net BOOT0: now reaches C9.2
- net BOOT0: now also IC1.44 (BOOT0), R3.1, SW3.1 (A)
- net PA0: now reaches R1.1
- net VDDRF: no longer names the net of C10.1
- net VDDRF: now also IC1.22 (VCAP1)
- new net: D2.2 (A), R6.2
- new net: FB1.2, IC1.9 (VDDA/VREF+)
- new net: D1.2 (A), R5.2
- new net: R1.2, SW1.1 (A)
- new net +3.3V: C1.1, C2.1, C3.1, FB1.1, IC1.1 (VBAT), IC1.24 (VDD_1), IC1.36 (VDD_2), IC1.48 (VDD_3), J1.1 (Pin_1), J3.2 (Pin_2), R2.2, R5.1, R6.1, SW3.2 (B)
- new net PA14: IC1.37 (PA14), J1.3 (Pin_3)
- new net PB2: IC1.20 (PB2), R4.1
- new net USB_D+: IC1.33 (PA12)
- new net USB_D-: IC1.32 (PA11)
- new net VREF+: C4.1, C5.1
- no-connect marks 1 -> 17
Other:
- note added: "BOOT Settings"
- note added: "EPS Power supply"
- note added: "Indicator light"
- note added: "Power supply"
- note added: "Reset circuit"
- note added: "SW debug download interface"
- note added: "User KEY"
- moved on the sheet: C6, C7, Y2
