File: payload1_board/rf.kicad_sch (KiCad schematic)
At the start: 25 parts, among them J4 Conn_Coaxial, U2 CG2179M2

Commit message: LAST UPDATE
Parts:
- U2: footprint MINISO6_CG21_CEL -> (none)
Connections:
- net PA13: no longer names the net of C35.2, U2.4 (VC2)
Changed lines of the file:
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@@
+		)
+	)
+	(text_box "Falta 1 GPIO\n"
+		(exclude_from_sim no)
+		(at 224.79 76.2 0)
+		(size 10.16 5.08)
+		(margins 0.9525 0.9525 0.9525 0.9525)
+		(stroke
+			(width 0)
+			(type solid)
+		)
+		(fill
+			(type none)
+		)
+		(effects
+			(font
+				(size 1.27 1.27)
+			)
+			(justify left top)
 		)
 	)
@@
 	)
 	(junction
+		(at 67.564 59.69)
+		(diameter 0)
+		(color 0 0 0 0)
+	)
+	(junction
 		(at 238.76 73.66)
 		(diameter 0)
@@
 	(wire
 		(pts
+			(xy 67.564 59.69) (xy 68.58 59.69)
+		)
+		(stroke
+			(width 0)
+			(type default)
+		)
+	)
+	(wire
+		(pts
 			(xy 78.74 110.49) (xy 63.5 110.49)
 		)
@@
 	(wire
 		(pts
-			(xy 63.5 59.69) (xy 68.58 59.69)
+			(xy 63.5 59.69) (xy 67.564 59.69)
 		)
 		(stroke
@@
 		)
 	)
-	(global_label "PA13"
-		(shape input)
-		(at 223.52 78.74 0)
-		(fields_autoplaced yes)
-		(effects
-			(font
-				(size 1.27 1.27)
-			)
-			(justify left)
-		)
-		(property "Intersheetrefs" "${INTERSHEET_REFS}"
-			(at 231.2828 78.74 0)
-			(effects
-				(font
-					(size 1.27 1.27)
-				)
-				(justify left)
-				(hide yes)
-			)
-		)
-	)
 	(global_label "RFO_HP"
 		(shape input)
@@
 	)
 	(symbol
+		(lib_id "power:PWR_FLAG")
+		(at 67.564 59.69 0)
+		(unit 1)
+		(exclude_from_sim no)
+		(in_bom yes)
+		(on_board yes)
+		(dnp no)
+		(fields_autoplaced yes)
+		(property "Reference" "#FLG06"
+			(at 67.564 57.785 0)
+			(effects
+				(font
+					(size 1.27 1.27)
+				)
+				(hide yes)
+			)
+		)
+		(property "Value" "PWR_FLAG"
+			(at 67.564 54.61 0)
+			(effects
+				(font
+					(size 1.27 1.27)
+				)
+			)
+		)
+		(property "Footprint" ""
+			(at 67.564 59.69 0)
+			(effects
+				(font
+					(size 1.27 1.27)
+				)
+				(hide yes)
+			)
+		)
+		(property "Datasheet" "~"
+			(at 67.564 59.69 0)
+			(effects
+				(font
+					(size 1.27 1.27)
+				)
+				(hide yes)
+			)
+		)
+		(property "Description" "Special symbol for telling ERC where power comes from"
+			(at 67.564 59.69 0)
+			(effects
+				(font
+					(size 1.27 1.27)
+				)
+				(hide yes)
+			)
+		)
+		(pin "1"
+		)
+		(instances
+			(project ""
+				(path "/ea597178-b44d-4db9-826c-8f86e8d231f0/f2ec5e10-3e2b-4fad-b66b-c622a3150eea"
+					(reference "#FLG06")
+					(unit 1)
+				)
+			)
+		)
+	)
+	(symbol
 		(lib_id "Device:L")
 		(at 87.63 86.36 90)
@@
 			)
 		)
-		(property "Footprint" "MINISO6_CG21_CEL"
+		(property "Footprint" ""
 			(at 194.564 85.09 0)
 			(effects
@@
 			)
 		)
-		(property "Datasheet" "CG2179M2"
+		(property "Datasheet" ""
 			(at 194.056 83.312 0)
 			(effects
