File: payload1_board/payload1_board.kicad_sch (KiCad schematic)
At the start: 0 parts

Commit message: a
Other:
- added sheet OCP (ocp.kicad_sch)
Changed lines of the file:
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@@
+	)
+	(sheet
+		(at 30.988 68.326)
+		(size 41.402 21.082)
+		(exclude_from_sim no)
+		(in_bom yes)
+		(on_board yes)
+		(dnp no)
+		(fields_autoplaced yes)
+		(stroke
+			(width 0.1524)
+			(type solid)
+		)
+		(fill
+			(color 0 0 0 0.0000)
+		)
+		(property "Sheetname" "OCP"
+			(at 30.988 67.6144 0)
+			(effects
+				(font
+					(size 1.27 1.27)
+				)
+				(justify left bottom)
+			)
+		)
+		(property "Sheetfile" "ocp.kicad_sch"
+			(at 30.988 89.9926 0)
+			(effects
+				(font
+					(size 1.27 1.27)
+				)
+				(justify left top)
+			)
+		)
+		(instances
+			(project "payload1_board"
+				(path "/ea597178-b44d-4db9-826c-8f86e8d231f0"
+					(page "6")
+				)
+			)
+		)
 	)
 	(sheet

Commit message: LAST UPDATE
Other:
- removed sheet GPS
- removed sheet RF
- added sheet IO_CONN (io_conn.kicad_sch)
Changed lines of the file:
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@@
 	(generator_version "9.0")
 	(paper "A4")
-	(text_box "GPS: MAX-M10S"
-		(exclude_from_sim no)
-		(at 135.89 55.88 0)
-		(size 33.02 6.35)
-		(margins 0.9525 0.9525 0.9525 0.9525)
-		(stroke
-			(width 0)
-			(type solid)
-		)
-		(fill
-			(type none)
-		)
-		(effects
-			(font
-				(size 1.27 1.27)
-			)
-			(justify left top)
-		)
-	)
-	(text_box "IMU: acelerometro, magnetometro y giroscopio"
-		(exclude_from_sim no)
-		(at 186.69 55.88 0)
-		(size 35.56 6.35)
-		(margins 0.9525 0.9525 0.9525 0.9525)
-		(stroke
-			(width 0)
-			(type solid)
-		)
-		(fill
-			(type none)
-		)
-		(effects
-			(font
-				(size 1.27 1.27)
-			)
-			(justify left top)
-		)
-	)
 	(sheet
-		(at 185.42 31.75)
+		(at 133.858 31.496)
 		(size 39.37 21.59)
 		(exclude_from_sim no)
@@
 		)
 		(property "Sheetname" "Sensores"
-			(at 185.42 31.0384 0)
+			(at 133.858 30.7844 0)
 			(effects
 				(font
@@
 		)
 		(property "Sheetfile" "sensores.kicad_sch"
-			(at 185.42 53.9246 0)
+			(at 133.858 53.6706 0)
 			(effects
 				(font
@@
 	)
 	(sheet
-		(at 135.89 31.75)
-		(size 34.29 21.59)
+		(at 181.61 31.242)
+		(size 44.958 21.082)
 		(exclude_from_sim no)
 		(in_bom yes)
@@
 			(color 0 0 0 0.0000)
 		)
-		(property "Sheetname" "GPS"
-			(at 135.89 31.0384 0)
+		(property "Sheetname" "IO_CONN"
+			(at 181.61 30.5304 0)
 			(effects
 				(font
@@
 			)
 		)
-		(property "Sheetfile" "gps.kicad_sch"
-			(at 135.89 53.9246 0)
+		(property "Sheetfile" "io_conn.kicad_sch"
+			(at 181.61 52.9086 0)
 			(effects
 				(font
@@
 			(project "payload1_board"
 				(path "/ea597178-b44d-4db9-826c-8f86e8d231f0"
-					(page "4")
+					(page "5")
 				)
 			)
@@
 	)
 	(sheet
-		(at 30.988 68.326)
+		(at 82.296 31.496)
 		(size 41.402 21.082)
 		(exclude_from_sim no)
@@
 		)
 		(property "Sheetname" "OCP"
-			(at 30.988 67.6144 0)
+			(at 82.296 30.7844 0)
 			(effects
 				(font
@@
 		)
 		(property "Sheetfile" "ocp.kicad_sch"
-			(at 30.988 89.9926 0)
+			(at 82.296 53.1626 0)
 			(effects
 				(font
@@
 				)
 			)
-		)
-	)
-	(sheet
-		(at 81.28 31.75)
-		(size 41.91 21.59)
-		(exclude_from_sim no)
-		(in_bom yes)
-		(on_board yes)
-		(dnp no)
-		(fields_autoplaced yes)
-		(stroke
-			(width 0.1524)
-			(type solid)
-		)
-		(fill
-			(color 0 0 0 0.0000)
-		)
-		(property "Sheetname" "RF"
-			(at 81.28 31.0384 0)
-			(effects
-				(font
-					(size 1.27 1.27)
-				)
-				(justify left bottom)
-			)
-		)
-		(property "Sheetfile" "rf.kicad_sch"
-			(at 81.28 53.9246 0)
-			(effects
-				(font
-					(size 1.27 1.27)
-				)
-				(justify left top)
-			)
-		)
-		(instances
-			(project "payload1_board"
-				(path "/ea597178-b44d-4db9-826c-8f86e8d231f0"
-					(page "3")
-				)
-			)

Commit message: update
Other:
- company: (none) -> Sanie Peralta, Alejandro Campo
- title: (none) -> Payload 2nd stage
Changed lines of the file:
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@@
 	(generator_version "9.0")
 	(paper "A4")
+	(title_block
+		(title "Payload 2nd stage")
+		(date "01/04/2026")
+		(company "Sanie Peralta, Alejandro Campo")
+	)
 	(sheet
 		(at 133.858 31.496)
